File: pcb/superenv/superenv.kicad_sch (KiCad schematic)
At the start: 31 parts, among them J1 TYPE-C-31-M-04, J10 PMSBB, J2 Power-Header, J3 UART0, J4 I2C, J5 I2C, J6 SGP41BB, J7 SCD41BB, J8 AHT20+BMP280BB, J9 UART1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

Commit message: Update gitignore and finish v1
Parts:
- removed C3: 4.7n, Capacitor_SMD:C_0402_1005Metric, symbol Device:C
- removed U5: DS18B20, Package_TO_SOT_THT:TO-92_Inline, symbol Sensor_Temperature:DS18B20
- added C4: 100n, Capacitor_SMD:C_0603_1608Metric, symbol Device:C
- added J11: DS18B20, Connector_PinHeader_2.54mm:PinHeader_1x03_P2.54mm_Vertical, symbol Connector_Generic:Conn_01x03
- added J12: GPIO, Connector_PinHeader_2.54mm:PinHeader_1x08_P2.54mm_Vertical, symbol Connector_Generic:Conn_01x08
- added J13: 3V3 rail, Connector_PinHeader_2.54mm:PinHeader_1x04_P2.54mm_Vertical, symbol Connector_Generic:Conn_01x04
- added J14: GND rail, Connector_PinHeader_2.54mm:PinHeader_1x04_P2.54mm_Vertical, symbol Connector_Generic:Conn_01x04
- added R8, R9: 10k, Resistor_SMD:R_0603_1608Metric, symbol Device:R
- C1: footprint Capacitor_SMD:C_0402_1005Metric -> Capacitor_SMD:C_0603_1608Metric; MFR CL05A105KA5NQNC -> CL10A105KB8NNNC
- C3: renamed from C4; footprint Capacitor_SMD:C_0402_1005Metric -> Capacitor_SMD:C_0603_1608Metric; MFR CL05B104KO5NNNC -> CC0603KRX7R9BB104
- C7: value 100n -> 4.7n; footprint Capacitor_SMD:C_0402_1005Metric -> Capacitor_SMD:C_0603_1608Metric; MFR CL05B104KO5NNNC -> 0603B472K500NT
- R1: footprint Resistor_SMD:R_0402_1005Metric -> Resistor_SMD:R_0603_1608Metric; MFR 0402WGF1004TCE -> 0603WAF1004T5E
- R2, R3: footprint Resistor_SMD:R_0402_1005Metric -> Resistor_SMD:R_0603_1608Metric; MFR 0402WGF5101TCE -> 0603WAF5101T5E
- R4: footprint Resistor_SMD:R_0402_1005Metric -> Resistor_SMD:R_0603_1608Metric; MFR 0402WGF1002TCE -> 0603WAF1002T5E
- R5, R6, R7: footprint Resistor_SMD:R_0402_1005Metric -> Resistor_SMD:R_0603_1608Metric; MFR 0402WGF4701TCE -> 0603WAF4701T5E
Connections:
- net +3V3: now also R6.2, R7.2, J11.3 (Pin_3), J13.1 (Pin_1), J13.2 (Pin_2), J13.3 (Pin_3), J13.4 (Pin_4), R8.1, R9.2; no longer R6.1, R7.1
- net +5V: now also J10.1 (Pin_1)
- net BOOT: now also C4.1; no longer C7.1
- net DQ: now also J11.2 (Pin_2)
- net GND: now also J10.2 (Pin_2), C4.2, J11.1 (Pin_1), J12.1 (Pin_1), J14.1 (Pin_1), J14.2 (Pin_2), J14.3 (Pin_3), J14.4 (Pin_4)
- net RXD_0: now also J10.5 (Pin_5)
- net SCL: now also R6.1; no longer R6.2
- net SDA: now also R7.1; no longer R7.2
- net TXD_0: now also J10.4 (Pin_4)
- net SET: now reaches U1.11 (GPIO10)
- net SET: now also J10.3 (Pin_3), R9.1
- net RST: now reaches U1.12 (GPIO11)
- net RST: now also J10.6 (Pin_6), R8.2
- net GPIO20: now reaches U1.18 (GPIO20)
- net GPIO20: now also J12.6 (Pin_6)
- net GPIO21: now reaches U1.19 (GPIO21)
- net GPIO21: now also J12.7 (Pin_7)
- net GPIO22: now reaches U1.20 (GPIO22)
- net GPIO22: now also J12.8 (Pin_8)
- net GPIO4: now reaches U1.4 (MTMS/GPIO4/ADC1_CH4)
- net GPIO4: now also J12.2 (Pin_2)
- net GPIO5: now reaches U1.5 (MTDI/GPIO5/ADC1_CH5)
- net GPIO5: now also J12.3 (Pin_3)
- net GPIO6: now reaches U1.6 (MTCK/GPIO6/ADC1_CH6)
- net GPIO6: now also J12.4 (Pin_4)
- net GPIO7: now reaches U1.7 (MTDO/GPIO7)
- net GPIO7: now also J12.5 (Pin_5)
- net at J1.S1 (SHIELD), R1.2: now also C7.1
- no-connect marks 3 -> 5
Other:
- moved on the sheet: J10, J3, J4, J5, J9, R4, U4
